File: base-station.kicad_pcb (KiCad board)
At the start: 2 copper layers, 85.7 x 87.2 mm, 68 parts, among them IC1 ATMEGA32-A, P1 HC-05, P2 NRF24L01+, P3 SERIAL, P4 LCD1, P5 LCD2, P6 POWER, Q1 BTEN, SW1 RESET, U1 LP5907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

Commit message: Added UCF logo
Parts:
- added G***: LOGO, LOGO, B.Cu at (133.0, 138.3)
