File: base-station.kicad_pcb (KiCad board)
At the start: 2 copper layers, 85.7 x 87.2 mm, 69 parts, among them IC1 ATMEGA32-A, P1 HC-05, P2 NRF24L01+, P3 SERIAL, P4 LCD1, P5 LCD2, P6 POWER, Q1 BTEN, SW1 RESET, U1 LP5907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

Commit message: Fix ISP SilkS bug and revision bump
Other:
- board text added: "Rev. 1.1"
- board text removed: "Rev. 1.0"
Changed lines of the file:
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@@
     )
   )
-  (module LOGO (layer B.Cu)
+  (module LOGO   locked (layer B.Cu)
     (at 132.969 138.303)
     (fp_text reference G*** (at 0 -20.91182) (layer B.SilkS) hide
@@
     (effects (font (size 1.5 1.5) (thickness 0.3)))
   )
-  (gr_text "Rev. 1.0" (at 161.163 81.407) (layer F.SilkS)
+  (gr_text "Rev. 1.1" (at 161.163 81.407) (layer F.SilkS)
     (effects (font (size 1.5 1.5) (thickness 0.3)))
   )
@@
   )
   (gr_line (start 163.83 151.257) (end 163.83 153.797) (angle 90) (layer F.SilkS) (width 0.2))
-  (gr_text RST (at 167.767 145.542 90) (layer F.SilkS)
+  (gr_text GND (at 167.767 145.161 90) (layer F.SilkS)
     (effects (font (size 1.016 1.016) (thickness 0.254)) (justify right))
   )
